File: DC-DC Module Board Mk.2.sch (EAGLE design)
At the start: 159 parts, among them Q1 FDN340P, U2 AP1117_LIN_REG, U3 LM1085IS-5.0

Commit message: final drcing
Parts:
- added C13: 0.1uF, rcl:C-USC0603
Connections:
- net +3V3: now also C13.1
- net DGND: now also C13.2
Changed lines of the file:
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@@
 <part name="R24" library="resistor" deviceset="R-US_" device="R0603" value="330"/>
 <part name="U3" library="NSC_By_element14_Batch_1" deviceset="LM1085IS-5.0" device=""/>
-<part name="5V_GND" library="supply2" deviceset="GND" device=""/>
 <part name="D10" library="diode" deviceset="BAS40" device=""/>
 <part name="C29" library="resistor" deviceset="C-EU" device="C0603" value="0.1u"/>
@@
 <part name="GND9" library="SparkFun-Aesthetics" deviceset="GND" device=""/>
 <part name="D1" library="SparkFun-LED" deviceset="LED-RED" device="0603" value="RED"/>
+<part name="GND14" library="SparkFun-Aesthetics" deviceset="GND" device=""/>
+<part name="C13" library="rcl" deviceset="C-US" device="C0603" value="0.1uF"/>
 </parts>
 <sheets>
@@
 <text x="40.64" y="-76.2" size="1.778" layer="95">One for each VDD</text>
 <text x="10.16" y="-73.66" size="1.778" layer="95">Conect to any one VDD</text>
-<wire x1="459.74" y1="-68.58" x2="533.4" y2="-68.58" width="0.1524" layer="97" style="shortdash"/>
+<wire x1="447.04" y1="-68.58" x2="533.4" y2="-68.58" width="0.1524" layer="97" style="shortdash"/>
 <wire x1="533.4" y1="-68.58" x2="533.4" y2="-127" width="0.1524" layer="97" style="shortdash"/>
-<wire x1="533.4" y1="-127" x2="459.74" y2="-127" width="0.1524" layer="97" style="shortdash"/>
-<wire x1="459.74" y1="-127" x2="459.74" y2="-68.58" width="0.1524" layer="97" style="shortdash"/>
+<wire x1="533.4" y1="-127" x2="447.04" y2="-127" width="0.1524" layer="97" style="shortdash"/>
+<wire x1="447.04" y1="-127" x2="447.04" y2="-68.58" width="0.1524" layer="97" style="shortdash"/>
 <text x="487.68" y="-66.04" size="1.778" layer="97">Yes we CAN!</text>
 <wire x1="218.44" y1="-165.1" x2="147.32" y2="-165.1" width="0.1524" layer="95" style="shortdash"/>
@@
 <instance part="R24" gate="G$1" x="408.94" y="-172.72" rot="MR90"/>
 <instance part="U3" gate="A" x="368.3" y="-160.02"/>
-<instance part="5V_GND" gate="GND" x="347.98" y="-170.18"/>
 <instance part="D10" gate="1" x="370.84" y="-147.32" rot="MR0"/>
 <instance part="C29" gate="G$1" x="403.86" y="-165.1" rot="R180"/>
@@
 </instance>
 <instance part="D1" gate="G$1" x="114.3" y="-144.78"/>
+<instance part="GND14" gate="1" x="347.98" y="-177.8" smashed="yes">
+<attribute name="VALUE" x="345.44" y="-180.34" size="1.778" layer="96"/>
+</instance>
+<instance part="C13" gate="G$1" x="452.12" y="-96.52"/>
 </instances>
 <busses>
@@
 <label x="396.24" y="73.66" size="1.27" layer="95" xref="yes"/>
 <label x="396.24" y="73.66" size="1.27" layer="95" xref="yes"/>
-</segment>
-<segment>
-<pinref part="U3" gate="A" pin="ADJ/GND"/>
-<pinref part="5V_GND" gate="GND" pin="GND"/>
-<wire x1="347.98" y1="-167.64" x2="347.98" y2="-165.1" width="0.1524" layer="91"/>
 </segment>
 <segment>
@@
 <wire x1="408.94" y1="-187.96" x2="408.94" y2="-193.04" width="0.1524" layer="91"/>
 <pinref part="GND9" gate="1" pin="GND"/>
+</segment>
+<segment>
+<pinref part="U3" gate="A" pin="ADJ/GND"/>
+<pinref part="GND14" gate="1" pin="GND"/>
+<wire x1="347.98" y1="-165.1" x2="347.98" y2="-175.26" width="0.1524" layer="91"/>
 </segment>
 </net>
@@
 <pinref part="U$8" gate="G$1" pin="GND"/>
 <wire x1="482.6" y1="-106.68" x2="480.06" y2="-106.68" width="0.1524" layer="91"/>
-<wire x1="480.06" y1="-106.68" x2="480.06" y2="-119.38" width="0.1524" layer="91"/>
+<wire x1="480.06" y1="-106.68" x2="480.06" y2="-114.3" width="0.1524" layer="91"/>
 <label x="480.06" y="-116.84" size="1.778" layer="95"/>
+<pinref part="C13" gate="G$1" pin="2"/>
+<wire x1="480.06" y1="-114.3" x2="480.06" y2="-119.38" width="0.1524" layer="91"/>
+<wire x1="452.12" y1="-101.6" x2="452.12" y2="-114.3" width="0.1524" layer="91"/>
+<wire x1="452.12" y1="-114.3" x2="480.06" y2="-114.3" width="0.1524" layer="91"/>
+<junction x="480.06" y="-114.3"/>
 </segment>
 <segment>
@@
 <wire x1="482.6" y1="-91.44" x2="480.06" y2="-91.44" width="0.1524" layer="91"/>
 <pinref part="+3V6" gate="G$1" pin="+3V3"/>
-<wire x1="480.06" y1="-76.2" x2="480.06" y2="-91.44" width="0.1524" layer="91"/>
-</segment>
-<segment>
+<wire x1="480.06" y1="-76.2" x2="480.06" y2="-81.28" width="0.1524" layer="91"/>
+<pinref part="C13" gate="G$1" pin="1"/>
+<wire x1="480.06" y1="-81.28" x2="480.06" y2="-91.44" width="0.1524" layer="91"/>
+<wire x1="480.06" y1="-81.28" x2="452.12" y2="-81.28" width="0.1524" layer="91"/>
+<wire x1="452.12" y1="-81.28" x2="452.12" y2="-93.98" width="0.1524" layer="91"/>
+<junction x="480.06" y="-81.28"/>
+</segment>
+<segment>
